File: JKP/JKP.kicad_pcb (KiCad board)
At the start: 2 copper layers, 366.7 x 119.1 mm, 225 parts, among them J1 Conn_01x04_Male, SW1 SW_Push, U1 ATmega32U4-AU, Y1 16MHz

Commit message: routing pcb part 1
Parts:
- added MX97: MX-NoLED, MX_Alps_Hybrid:MX-1.5U-NoLED, F.Cu at (4.76, 57.1)
- C1, C2, C3, C4, C5, C6, C7, D1, D10, D100, D101, D102, D103, D104, D105, D106, D107, D108, D109, D11, D110, D111, D112, D12, D13, D14, D15, D16, D17, D18, D19, D2, D20, D21, D22, D23, D24, D25, D26, D27, D28, D29, D3, D30, D31, D32, D33, D34, D35, D36, D37, D38, D39, D4, D40, D41, D42, D43, D44, D45, D46, D47, D48, D49, D5, D50, D51, D52, D53, D54, D55, D56, D57, D58, D59, D6, D60, D61, D62, D63, D64, D65, D66, D67, D68, D69, D7, D70, D71, D72, D73, D74, D75, D76, D77, D78, D79, D8, D80, D81, D82, D83, D84, D85, D86, D87, D88, D89, D9, D90, D91, D92, D93, D94, D95, D96, D97, D98, D99, F1, J1, R1, R2, R3, R4, R5, SW1, U1, Y1: moved to B.Cu
- moved D1 459.6 mm to (350.8, -19.0), turned to 90 degrees
- moved D96 444.7 mm to (307.2, 90.5), turned to 180 degrees
- moved D98 443.8 mm to (319.1, 14.3), turned to 180 degrees
- moved D2 442.5 mm to (342.1, -19.8), turned to 270 degrees
- moved U1 427.4 mm to (275.4, 57.1), turned to 180 degrees
- moved D95 426.6 mm to (300.0, 71.4), turned to 180 degrees
- moved C3 423.0 mm to (273.1, 71.4), turned to 270 degrees
- moved C1 422.2 mm to (269.9, 47.6)
- moved D94 415.9 mm to (300.0, 52.4), turned to 180 degrees
- moved C2 415.4 mm to (263.5, 61.9), turned to 270 degrees
- moved D86 399.4 mm to (257.3, 61.9), turned to 90 degrees
- moved D3 394.5 mm to (328.6, -25.4), turned to 270 degrees
- moved D105 392.8 mm to (338.1, 52.4), turned to 180 degrees
- moved D103 389.0 mm to (338.1, 14.3), turned to 180 degrees
- moved C6 387.1 mm to (281.0, 47.6), turned to 180 degrees
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Connections:
- D1 pad 1: Net-(D1-Pad1) -> +5V
- D1 pad 3: Net-(D1-Pad3) -> GND
- D112 pad 1: ROW4 -> ROW5
- D14 pad 1: Net-(D14-Pad1) -> +5V
- D14 pad 3: Net-(D14-Pad3) -> GND
- D2 pad 1: Net-(D2-Pad1) -> +5V
- D2 pad 3: Net-(D2-Pad3) -> GND
- D27 pad 1: Net-(D27-Pad1) -> +5V
- D27 pad 3: Net-(D27-Pad3) -> GND
- D3 pad 1: Net-(D3-Pad1) -> +5V
- D3 pad 3: Net-(D3-Pad3) -> GND
- D33 pad 1: Net-(D33-Pad1) -> +5V
- D33 pad 3: Net-(D33-Pad3) -> GND
- D39 pad 1: Net-(D39-Pad1) -> +5V
- D39 pad 3: Net-(D39-Pad3) -> GND
- D4 pad 1: Net-(D4-Pad1) -> +5V
- D4 pad 3: Net-(D4-Pad3) -> GND
- D45 pad 1: Net-(D45-Pad1) -> +5V
- D45 pad 3: Net-(D45-Pad3) -> GND
- D5 pad 1: Net-(D5-Pad1) -> +5V
- D5 pad 3: Net-(D5-Pad3) -> GND
- D52 pad 1: Net-(D52-Pad1) -> +5V
- D52 pad 3: Net-(D52-Pad3) -> GND
- D58 pad 1: Net-(D58-Pad1) -> +5V
- D58 pad 3: Net-(D58-Pad3) -> GND
- D6 pad 1: Net-(D6-Pad1) -> +5V
- D6 pad 3: Net-(D6-Pad3) -> GND
- D64 pad 1: Net-(D64-Pad1) -> +5V
- D64 pad 3: Net-(D64-Pad3) -> GND
- D7 pad 1: Net-(D7-Pad1) -> +5V
- D7 pad 3: Net-(D7-Pad3) -> GND
- D70 pad 1: Net-(D70-Pad1) -> +5V
- D70 pad 3: Net-(D70-Pad3) -> GND
- MX29 pad 1: COL5 -> COL6
- MX34 pad 1: COL6 -> COL7
- MX40 pad 1: COL7 -> COL8
- MX45 pad 1: COL8 -> COL9
- MX50 pad 1: COL9 -> COL10
- MX55 pad 1: COL10 -> COL11
- MX61 pad 1: COL11 -> COL12
- MX67 pad 1: COL12 -> COL13
- MX80 pad 1: COL14 -> COL15
Routing:
- net ROW1: track 0.00 -> 395.1 mm, vias 0 -> 2
- net ROW2: track 0.00 -> 390.3 mm, vias 0 -> 2
- net ROW0: track 0.00 -> 380.8 mm
- net ROW4: track 0.00 -> 372.2 mm
- net ROW5: track 0.00 -> 351.7 mm
- net ROW3: track 0.00 -> 344.3 mm
- net COL12: track 0.00 -> 143.2 mm
- net COL11: track 0.00 -> 134.6 mm
- net COL10: track 0.00 -> 131.2 mm
- net COL1: track 0.00 -> 127.5 mm
- net COL0: track 0.00 -> 127.4 mm
- net COL2: track 0.00 -> 123.5 mm
- net COL6: track 0.00 -> 119.2 mm
- net COL3: track 0.00 -> 103.6 mm
- net COL4: track 0.00 -> 103.1 mm
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Other:
- board size 366.7 x 119.1 mm -> 366.7 x 114.3 mm
- net class Power added: clearance 0.2, trace_width 0.381, via_dia 0.8, via_drill 0.4

Commit message: Finished PCB v1 No LED
Parts:
- removed D1, D14, D2, D27, D3, D33, D39, D4, D45, D5, D52, D58, D6, D64, D7, D70: WS2812B, LED_SMD:LED_WS2812B_PLCC4_5.0x5.0mm_P3.2mm
- removed R1: 500 ohms, Resistor_SMD:R_0805_2012Metric
- moved R4 285.8 mm to (283.4, 71.6), turned to 270 degrees
- moved R5 265.8 mm to (263.8, 51.1), turned to 270 degrees
- moved SW1 213.3 mm to (278.6, 82.5), turned to 270 degrees
- moved D86 13.2 mm to (255.7, 48.8), turned to 0 degrees
- moved C2 1.12 mm to (264.3, 61.1), turned to 0 degrees
- moved C7 0.72 mm to (287.4, 59.6), turned to 90 degrees
Connections:
- U1 pad 1: Net-(U1-Pad1) -> COL14
- U1 pad 10: Net-(U1-Pad10) -> COL17
- U1 pad 11: Net-(U1-Pad11) -> ROW3
- U1 pad 12: Net-(U1-Pad12) -> ROW5
- U1 pad 18: Net-(U1-Pad18) -> COL12
- U1 pad 19: Net-(U1-Pad19) -> ROW4
- U1 pad 20: Net-(U1-Pad20) -> COL0
- U1 pad 21: Net-(U1-Pad21) -> COL1
- U1 pad 22: Net-(U1-Pad22) -> COL2
- U1 pad 25: Net-(U1-Pad25) -> COL3
- U1 pad 26: Net-(U1-Pad26) -> COL4
- U1 pad 27: Net-(U1-Pad27) -> COL5
- U1 pad 28: Net-(U1-Pad28) -> COL6
- U1 pad 29: Net-(U1-Pad29) -> COL7
- U1 pad 30: Net-(U1-Pad30) -> COL8
- U1 pad 31: Net-(U1-Pad31) -> COL9
- U1 pad 36: Net-(U1-Pad36) -> COL10
- U1 pad 37: Net-(U1-Pad37) -> COL11
- U1 pad 38: Net-(U1-Pad38) -> COL13
- U1 pad 39: Net-(U1-Pad39) -> ROW2
- U1 pad 40: Net-(U1-Pad40) -> ROW1
- U1 pad 41: Net-(U1-Pad41) -> ROW0
- U1 pad 8: Net-(U1-Pad8) -> COL15
- U1 pad 9: Net-(U1-Pad9) -> COL16
Routing:
- net COL0: track 127.4 -> 422.2 mm
- net COL1: track 127.5 -> 387.5 mm
- net COL2: track 123.5 -> 352.7 mm
- net COL3: track 103.6 -> 314.2 mm
- net COL4: track 103.1 -> 294.3 mm
- net COL5: track 77.9 -> 249.3 mm
- net COL6: track 119.2 -> 271.6 mm
- net COL7: track 99.6 -> 247.4 mm
- net ROW3: track 344.3 -> 484.6 mm, vias 0 -> 2
- net COL8: track 100.2 -> 228.1 mm
- net COL9: track 100.2 -> 208.9 mm
- net +5V: track 50.6 -> 153.2 mm, vias 0 -> 5
- net COL10: track 131.2 -> 220.9 mm
- net ROW5: track 351.7 -> 441.4 mm
- net COL11: track 134.6 -> 205.9 mm
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
Commit message: double checking
Routing:
- added copper zone on B.Cu, net GND
- added copper zone on F.Cu, net GND

Commit message: changed PCB to screwless design
Parts:
- moved D15 6.35 mm to (38.1, 1.59)
- moved D40 6.35 mm to (128.6, 1.59)
- moved D65 6.35 mm to (219.1, 1.59)
- moved D71 6.35 mm to (238.1, 1.59)
Routing:
- net ROW0: track 435.8 -> 471.7 mm
- net Net-(D40-Pad2): track 5.48 -> 11.4 mm
- net Net-(D15-Pad2): track 5.48 -> 11.4 mm
- net Net-(D71-Pad2): track 5.48 -> 11.0 mm
- net Net-(D65-Pad2): track 5.48 -> 11.0 mm
- net COL2: track 352.7 -> 348.5 mm
- net COL9: track 208.9 -> 207.5 mm
- removed copper zone on B.Cu, net GND
- removed copper zone on F.Cu, net GND
Other:
- outline, holes or cut-outs redrawn

Commit message: screwless pcb cutouts
Routing:
- net COL12: track 162.6 -> 165.4 mm
- net ROW3: track 484.6 -> 483.2 mm
Other:
- outline, holes or cut-outs redrawn

Commit message: final PCB v1
Parts:
- MX65: footprint MX_Alps_Hybrid:MX-1.75U-NoLED -> MX_Alps_Hybrid:MX-1.5U-NoLED
Routing:
- net COL0: track 422.1 -> 417.7 mm
- net Net-(D11-Pad2): track 12.6 -> 14.2 mm
- added copper zone on B.Cu, net GND
- added copper zone on F.Cu, net GND
Other:
- outline, holes or cut-outs redrawn

Commit message: final PCB v1
Parts:
- renumbered D8 to D1, D18 to D10, D19 to D11, D20 to D12, D21 to D13, D22 to D14, D23 to D15, D24 to D16, D25 to D17, D26 to D18, D28 to D19, D9 to D2, D29 to D20, D30 to D21, D31 to D22, D32 to D23, D34 to D24, D35 to D25, D36 to D26, D37 to D27, D38 to D28, D41 to D29, D10 to D3, D42 to D30, D43 to D31, D44 to D32, D40 to D33, D47 to D34, D48 to D35, D49 to D36, D50 to D37, D51 to D38, D46 to D39, D11 to D4, D54 to D40, D55 to D41, D56 to D42, D57 to D43, D53 to D44, D60 to D45, D61 to D46, D62 to D47, D63 to D48, D59 to D49, D12 to D5, D66 to D50, D67 to D51, D68 to D52, D69 to D53, D65 to D54, D72 to D55, D73 to D56, D74 to D57, D75 to D58, D76 to D59, D13 to D6, D71 to D60, D78 to D61, D79 to D62, D80 to D63, D81 to D64, D82 to D65, D77 to D66, D84 to D67, D85 to D68, D86 to D69, D15 to D7, D87 to D70, D88 to D71, D83 to D72, D89 to D73, D90 to D74, D91 to D75, D92 to D76, D93 to D77, D94 to D78, D95 to D79, D16 to D8, D97 to D80, D98 to D81, D99 to D82, D100 to D83, D101 to D84, D96 to D85, D102 to D86, D103 to D87, D104 to D88, D105 to D89, D17 to D9, D106 to D90, D107 to D91, D108 to D92, D109 to D93, D110 to D94, D111 to D95, D112 to D96, MX97 to MX1, MX9 to MX10, MX10 to MX11, MX11 to MX12, MX12 to MX13, MX13 to MX14, MX14 to MX15, MX15 to MX16, MX16 to MX17, MX17 to MX18, MX18 to MX19, MX1 to MX2, MX19 to MX20, MX20 to MX21, MX21 to MX22, MX22 to MX23, MX23 to MX24, MX24 to MX25, MX25 to MX26, MX26 to MX27, MX27 to MX28, MX28 to MX29, MX2 to MX3, MX29 to MX34, MX3 to MX4, MX34 to MX40, MX40 to MX45, MX4 to MX5, MX45 to MX50, MX50 to MX55, MX5 to MX6, MX55 to MX61, MX61 to MX67, MX6 to MX7, MX67 to MX73, MX73 to MX74, MX74 to MX75, MX75 to MX76, MX76 to MX77, MX77 to MX78, MX78 to MX79, MX7 to MX8, MX79 to MX80, MX80 to MX86, MX86 to MX87, MX87 to MX88, MX88 to MX89, MX8 to MX9, MX89 to MX90, MX90 to MX91, MX91 to MX92, MX92 to MX93, MX93 to MX94, MX94 to MX95, MX95 to MX96, MX96 to MX97, R2 to R1, R3 to R2, R4 to R3, R5 to R4

Commit message: fixed VBUS not connected
Parts:
- F1: value Polyfuse_Small -> 500mA
- moved C7 0.33 mm to (287.5, 59.9)
Connections:
- U1 pad 7: Net-(U1-Pad7) -> +5V
Routing:
- net GND: track 99.9 -> 120.8 mm
- net ROW4: track 403.2 -> 408.1 mm
- net +5V: track 153.2 -> 155.7 mm, vias 5 -> 6
- net ROW5: track 441.4 -> 443.1 mm
- net COL17: track 163.5 -> 164.4 mm
- net COL15: track 128.5 -> 129.1 mm
- net COL16: track 146.2 -> 146.9 mm
